File: PCB/pixel-frame-adapter.kicad_pcb (KiCad board)
At the start: 2 copper layers, 38.3 x 41.9 mm, 4 parts, among them U1 Adafruit_1_54in_TFT, U2 Adafruit_ItsyBitsy_M4, U3 Adafruit_LIS3DH

Commit message: clean up
Connections:
- U1 pad 8: unconnected-(U1-Pad8) -> RST
- U2 pad 30: unconnected-(U2-Pad30) -> RST
Routing:
- net RST: track 0.00 -> 35.2 mm, vias 0 -> 2
Changed lines of the file:
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@@
   (net 6 "SD_CARD_MISO")
   (net 7 "SPI_MOSI")
-  (net 8 "unconnected-(U1-Pad8)")
+  (net 8 "RST")
   (net 9 "SPI_DC")
   (net 10 "SD_CARD_CS")
@@
   (net 32 "unconnected-(U2-Pad28)")
   (net 33 "unconnected-(U2-Pad29)")
-  (net 34 "unconnected-(U2-Pad30)")
-  (net 35 "unconnected-(U2-Pad31)")
-  (net 36 "unconnected-(U2-Pad33)")
-  (net 37 "unconnected-(U3-Pad1)")
-  (net 38 "unconnected-(U3-Pad2)")
-  (net 39 "unconnected-(U3-Pad3)")
-  (net 40 "unconnected-(U3-Pad4)")
-  (net 41 "unconnected-(U3-Pad5)")
-  (net 42 "unconnected-(U3-Pad8)")
-  (net 43 "Net-(JP1-Pad2)")
+  (net 34 "unconnected-(U2-Pad31)")
+  (net 35 "unconnected-(U2-Pad33)")
+  (net 36 "unconnected-(U3-Pad1)")
+  (net 37 "unconnected-(U3-Pad2)")
+  (net 38 "unconnected-(U3-Pad3)")
+  (net 39 "unconnected-(U3-Pad4)")
+  (net 40 "unconnected-(U3-Pad5)")
+  (net 41 "unconnected-(U3-Pad8)")
+  (net 42 "Net-(JP1-Pad2)")
   (footprint "pixel-frame-library:Adafruit_ItsyBitsy_M4" (layer "F.Cu")
     (at 160.9852 122.9106 180)
@@
       (net 33 "unconnected-(U2-Pad29)") (pinfunction "D12") (pintype "input+no_connect"))
     (pad "30" thru_hole circle (at 7.62 10.16 180) (size 1.524 1.524) (drill 0.762) (layers *.Cu *.Mask)
-      (net 34 "unconnected-(U2-Pad30)") (pinfunction "D13") (pintype "input+no_connect"))
+      (net 8 "RST") (pinfunction "D13") (pintype "input"))
     (pad "31" thru_hole circle (at 7.62 7.62 180) (size 1.524 1.524) (drill 0.762) (layers *.Cu *.Mask)
-      (net 35 "unconnected-(U2-Pad31)") (pinfunction "VBUS") (pintype "input+no_connect"))
+      (net 34 "unconnected-(U2-Pad31)") (pinfunction "VBUS") (pintype "input+no_connect"))
     (pad "32" thru_hole circle (at 7.62 5.08 180) (size 1.524 1.524) (drill 0.762) (layers *.Cu *.Mask)
       (net 4 "GND") (pinfunction "GND") (pintype "input"))
     (pad "33" thru_hole circle (at 7.62 2.54 180) (size 1.524 1.524) (drill 0.762) (layers *.Cu *.Mask)
-      (net 36 "unconnected-(U2-Pad33)") (pinfunction "VBAT") (pintype "input+no_connect"))
+      (net 35 "unconnected-(U2-Pad33)") (pinfunction "VBAT") (pintype "input+no_connect"))
   )
   (footprint "pixel-frame-library:Adafruit_LIS3DH" (layer "F.Cu")
@@
     (fp_rect (start -2.54 0) (end 15.24 22.86) (layer "Eco1.User") (width 0.12) (fill none))
     (pad "1" thru_hole circle (at 0 5.08 180) (size 1.524 1.524) (drill 0.762) (layers *.Cu *.Mask)
-      (net 37 "unconnected-(U3-Pad1)") (pinfunction "CS") (pintype "input+no_connect"))
+      (net 36 "unconnected-(U3-Pad1)") (pinfunction "CS") (pintype "input+no_connect"))
     (pad "2" thru_hole circle (at 0 7.62 180) (size 1.524 1.524) (drill 0.762) (layers *.Cu *.Mask)
-      (net 38 "unconnected-(U3-Pad2)") (pinfunction "SDO") (pintype "input+no_connect"))
+      (net 37 "unconnected-(U3-Pad2)") (pinfunction "SDO") (pintype "input+no_connect"))
     (pad "3" thru_hole circle (at 0 10.16 180) (size 1.524 1.524) (drill 0.762) (layers *.Cu *.Mask)
-      (net 39 "unconnected-(U3-Pad3)") (pinfunction "A1") (pintype "input+no_connect"))
+      (net 38 "unconnected-(U3-Pad3)") (pinfunction "A1") (pintype "input+no_connect"))
     (pad "4" thru_hole circle (at 0 12.7 180) (size 1.524 1.524) (drill 0.762) (layers *.Cu *.Mask)
-      (net 40 "unconnected-(U3-Pad4)") (pinfunction "A2") (pintype "input+no_connect"))
+      (net 39 "unconnected-(U3-Pad4)") (pinfunction "A2") (pintype "input+no_connect"))
     (pad "5" thru_hole circle (at 0 15.24 180) (size 1.524 1.524) (drill 0.762) (layers *.Cu *.Mask)
-      (net 41 "unconnected-(U3-Pad5)") (pinfunction "A3") (pintype "input+no_connect"))
+      (net 40 "unconnected-(U3-Pad5)") (pinfunction "A3") (pintype "input+no_connect"))
     (pad "6" thru_hole circle (at 0 17.78 180) (size 1.524 1.524) (drill 0.762) (layers *.Cu *.Mask)
       (net 25 "ACC_INT2") (pinfunction "INT_2") (pintype "input"))
@@
       (net 2 "+5V") (pinfunction "VIN") (pintype "input"))
     (pad "8" thru_hole circle (at 12.7 15.24 180) (size 1.524 1.524) (drill 0.762) (layers *.Cu *.Mask)
-      (net 42 "unconnected-(U3-Pad8)") (pinfunction "3V") (pintype "input+no_connect"))
+      (net 41 "unconnected-(U3-Pad8)") (pinfunction "3V") (pintype "input+no_connect"))
     (pad "9" thru_hole circle (at 12.7 12.7 180) (size 1.524 1.524) (drill 0.762) (layers *.Cu *.Mask)
       (net 4 "GND") (pinfunction "GND") (pintype "input"))
@@
       (net 31 "SPI_CS") (pinfunction "TC") (pintype "input"))
     (pad "8" thru_hole circle (at 0 22.86 180) (size 1.524 1.524) (drill 0.762) (layers *.Cu *.Mask)
-      (net 8 "unconnected-(U1-Pad8)") (pinfunction "RT") (pintype "input+no_connect"))
+      (net 8 "RST") (pinfunction "RT") (pintype "input"))
     (pad "9" thru_hole circle (at 0 25.4 180) (size 1.524 1.524) (drill 0.762) (layers *.Cu *.Mask)
       (net 9 "SPI_DC") (pinfunction "DC") (pintype "input"))
@@
       (net 10 "SD_CARD_CS") (pinfunction "CC") (pintype "input"))
     (pad "11" thru_hole circle (at 0 30.48 180) (size 1.524 1.524) (drill 0.762) (layers *.Cu *.Mask)
-      (net 43 "Net-(JP1-Pad2)") (pinfunction "BL") (pintype "input"))
+      (net 42 "Net-(JP1-Pad2)") (pinfunction "BL") (pintype "input"))
     (pad "12" thru_hole circle (at 0 33.02 180) (size 1.524 1.524) (drill 0.762) (layers *.Cu *.Mask)
       (net 11 "unconnected-(U1-Pad12)") (pinfunction "TE") (pintype "input+no_connect"))
@@
       ))
     (pad "2" smd custom (at 0.65 0 180) (size 1 0.5) (layers "F.Cu" "F.Mask")
-      (net 43 "Net-(JP1-Pad2)") (pinfunction "B") (pintype "passive") (zone_connect 2)
+      (net 42 "Net-(JP1-Pad2)") (pinfunction "B") (pintype "passive") (zone_connect 2)
       (options (clearance outline) (anchor rect))
       (primitives
@@
   (segment (start 134.467596 110.235996) (end 135.7122 111.4806) (width 0.2286) (layer "B.Cu") (net 7))
   (segment (start 155.6258 111.4806) (end 155.6258 93.6244) (width 0.2286) (layer "B.Cu") (net 7))
+  (segment (start 136.8552 98.171) (end 139.827 98.171) (width 0.2286) (layer "F.Cu") (net 8))
+  (segment (start 134.156196 98.171) (end 136.8552 98.171) (width 0.2286) (layer "F.Cu") (net 8))
+  (segment (start 132.8674 96.882204) (end 134.156196 98.171) (width 0.2286) (layer "F.Cu") (net 8))
+  (segment (start 140.462 112.7506) (end 140.1064 112.395) (width 0.2286) (layer "F.Cu") (net 8))
+  (segment (start 153.3652 112.7506) (end 140.462 112.7506) (width 0.2286) (layer "F.Cu") (net 8))
+  (via (at 139.827 98.171) (size 0.8128) (drill 0.4064) (layers "F.Cu" "B.Cu") (net 8))
+  (via (at 140.1064 112.395) (size 0.8128) (drill 0.4064) (layers "F.Cu" "B.Cu") (net 8))
+  (segment (start 140.1064 112.395) (end 140.1064 98.4504) (width 0.2286) (layer "B.Cu") (net 8))
+  (segment (start 140.1064 98.4504) (end 139.827 98.171) (width 0.2286) (layer "B.Cu") (net 8))
   (segment (start 134.130796 95.6056) (end 139.7508 95.6056) (width 0.2286) (layer "F.Cu") (net 9))
   (segment (start 139.7508 95.6056) (end 142.2908 98.1456) (width 0.2286) (layer "F.Cu") (net 9))
@@
   (via (at 147.0914 100.6094) (size 0.8128) (drill 0.4064) (layers "F.Cu" "B.Cu") (net 31))
   (segment (start 147.0914 100.6094) (end 147.0914 105.7656) (width 0.2286) (layer "B.Cu") (net 31))
-  (segment (start 135.375396 89.262204) (end 138.938 85.6996) (width 0.2286) (layer "F.Cu") (net 43))
-  (segment (start 132.8674 89.262204) (end 135.375396 89.262204) (width 0.2286) (layer "F.Cu") (net 43))
-  (segment (start 138.938 85.6996) (end 140.4724 85.6996) (width 0.2286) (layer "F.Cu") (net 43))
+  (segment (start 135.375396 89.262204) (end 138.938 85.6996) (width 0.2286) (layer "F.Cu") (net 42))
+  (segment (start 132.8674 89.262204) (end 135.375396 89.262204) (width 0.2286) (layer "F.Cu") (net 42))
+  (segment (start 138.938 85.6996) (end 140.4724 85.6996) (width 0.2286) (layer "F.Cu") (net 42))
   (zone (net 4) (net_name "GND") (layer "B.Cu") (hatch edge 0.508)
     (connect_pads (clearance 0.508))

Commit message: even numbers
Parts:
- moved U2 0.08 mm to (161.1, 122.9)
Routing:
- net SPI_MOSI: track 61.9 -> 60.6 mm
Other:
- board size 38.3 x 41.9 mm -> 38.4 x 41.9 mm
