File: PCB/pixel-frame-adapter.kicad_pcb (KiCad board)
At the start: 2 copper layers, 38.4 x 41.9 mm, 4 parts, among them U1 Adafruit_1_54in_TFT, U2 Adafruit_ItsyBitsy_M4, U3 Adafruit_LIS3DH

Commit message: handle through hole tolerances
Other:
- board text added: "V2.0"
- board text removed: "V1.0"
